Commit message: UPDATE:MELON

File: melon_ws/src/melon_description/urdf/base_v4.xacro (robot description, xacro)
@@ -18,8 +18,7 @@
         <inertia ixx="16.050446" iyy="13.982493" izz="18.567703" ixy="0.002034" iyz="-2.999695" ixz="0.007151"/>
       </inertial>
-      <visual>
+      <!-- <visual>
         <origin xyz="0 0 0" rpy="0 0 1.57"/>
         <geometry>
-          <!-- <mesh filename="file://$(find melon_description)/meshes/base_link.stl" scale="0.001 0.001 0.001"/> -->
           <mesh filename="package://melon_description/meshes/base_link.stl" scale="0.001 0.001 0.001"/>
         </geometry>
@@ -29,7 +28,98 @@
         <origin xyz="0 0 0" rpy="0 0 1.57"/>
         <geometry>
-          <!-- <mesh filename="file://$(find melon_description)/meshes/base_link.stl" scale="0.001 0.001 0.001"/> -->
           <mesh filename="package://melon_description/meshes/base_link.stl" scale="0.001 0.001 0.001"/>
-          <!-- <box size="0.715 0.82 0.42"/> -->
+        </geometry>
+      </collision> -->
+      <!-- body -->
+      <visual>
+        <origin xyz="-0.002 0.005 0.05" rpy="0 0 1.57"/>
+        <geometry>
+          <mesh filename="package://melon_description/meshes/body_1.stl" scale="0.001 0.001 0.001"/>
+        </geometry>
+        <material name="midnight_blue"/>
+      </visual>
+      <collision>
+        <origin xyz="-0.002 0.005 0.05" rpy="0 0 1.57"/>
+        <geometry>
+          <mesh filename="package://melon_description/meshes/body_1.stl" scale="0.001 0.001 0.001"/>
+        </geometry>
+      </collision>
+      <visual>
+        <origin xyz="0.0075 0.678 0.069" rpy="0 0 1.57"/>
+        <geometry>
+          <mesh filename="package://melon_description/meshes/body_2.stl" scale="0.001 0.001 0.001"/>
+        </geometry>
+        <material name="dark_black"/>
+      </visual>
+      <collision>
+        <origin xyz="0.0075 0.678 0.069" rpy="0 0 1.57"/>
+        <geometry>
+          <mesh filename="package://melon_description/meshes/body_2.stl" scale="0.001 0.001 0.001"/>
+        </geometry>
+      </collision>
+      <visual>
+        <origin xyz="0.027 0.025 0.37" rpy="0 0 -1.57"/>
+        <geometry>
+          <mesh filename="package://melon_description/meshes/body_3.stl" scale="0.001 0.001 0.001"/>
+        </geometry>
+        <material name="charcoal"/>
+      </visual>
+      <collision>
+        <origin xyz="0.027 0.025 0.37" rpy="0 0 -1.57"/>
+        <geometry>
+          <mesh filename="package://melon_description/meshes/body_3.stl" scale="0.001 0.001 0.001"/>
+        </geometry>
+      </collision>
+      <!-- caster mount -->
+      <visual>
+        <origin xyz="0.3 0.200 0.06" rpy="3.14 0 1.57"/>
+        <geometry>
+          <mesh filename="package://melon_description/meshes/ballfoint.stl" scale="0.001 0.001 0.001"/>
+        </geometry>
+        <material name="midnight_blue"/>
+      </visual>
+      <collision>
+        <origin xyz="0.3 0.200 0.06" rpy="3.14 0 1.57"/>
+        <geometry>
+          <mesh filename="package://melon_description/meshes/ballfoint.stl" scale="0.001 0.001 0.001"/>
+        </geometry>
+      </collision>
+      <visual>
+        <origin xyz="0.3 -0.200 0.06" rpy="3.14 0 1.57"/>
+        <geometry>
+          <mesh filename="package://melon_description/meshes/ballfoint.stl" scale="0.001 0.001 0.001"/>
+        </geometry>
+        <material name="midnight_blue"/>
+      </visual>
+      <collision>
+        <origin xyz="0.3 -0.200 0.06" rpy="3.14 0 1.57"/>
+        <geometry>
+          <mesh filename="package://melon_description/meshes/ballfoint.stl" scale="0.001 0.001 0.001"/>
+        </geometry>
+      </collision>
+      <visual>
+        <origin xyz="-0.33 0.200 0.06" rpy="3.14 0 1.57"/>
+        <geometry>
+          <mesh filename="package://melon_description/meshes/ballfoint.stl" scale="0.001 0.001 0.001"/>
+        </geometry>
+        <material name="midnight_blue"/>
+      </visual>
+      <collision>
+        <origin xyz="-0.33 0.200 0.06" rpy="3.14 0 1.57"/>
+        <geometry>
+          <mesh filename="package://melon_description/meshes/ballfoint.stl" scale="0.001 0.001 0.001"/>
+        </geometry>
+      </collision>
+      <visual>
+        <origin xyz="-0.33 -0.200 0.06" rpy="3.14 0 1.57"/>
+        <geometry>
+          <mesh filename="package://melon_description/meshes/ballfoint.stl" scale="0.001 0.001 0.001"/>
+        </geometry>
+        <material name="midnight_blue"/>
+      </visual>
+      <collision>
+        <origin xyz="-0.33 -0.200 0.06" rpy="3.14 0 1.57"/>
+        <geometry>
+          <mesh filename="package://melon_description/meshes/ballfoint.stl" scale="0.001 0.001 0.001"/>
         </geometry>
       </collision>
@@ -52,5 +142,4 @@
         <origin xyz="0.242002 0.007002 -0.10065" rpy="0 0 0"/>
         <geometry>
-          <!-- <mesh filename="file://$(find melon_description)/meshes/right_wheel_1.stl" scale="0.001 0.001 0.001"/> -->
           <mesh filename="package://melon_description/meshes/right_wheel_1.stl" scale="0.001 0.001 0.001"/>
         </geometry>
@@ -58,9 +147,6 @@
       </visual>
       <collision>
-        <origin xyz="-0.02 0.0 0.0" rpy="0 1.57 0"/>
-        <!-- <origin xyz="0.242002 0.007002 -0.10065" rpy="0 0 0"/> -->
-        <geometry>
-          <!-- <mesh filename="file://$(find melon_description)/meshes/right_wheel_1.stl" scale="0.001 0.001 0.001"/> -->
-          <!-- <mesh filename="package://melon_description/meshes/right_wheel_1.stl" scale="0.001 0.001 0.001"/> -->
+        <origin xyz="-0.04 0.0 0.0" rpy="0 1.57 0"/>
+        <geometry>
           <cylinder length="0.05" radius="0.10065"/>
         </geometry>
@@ -68,5 +154,5 @@
     </link>
     <joint name="${prefix}left_wheel_joint" type="continuous">
-      <origin xyz="0.007002 0.277998 0.10065" rpy="0 0 1.57"/>
+      <origin xyz="0.007002 0.279998 0.10065" rpy="0 0 1.57"/>
       <parent link="${prefix}base_link"/>
       <child link="${prefix}left_wheel_1"/>
@@ -83,5 +169,4 @@
         <origin xyz="-0.277998 0.007002 -0.10065" rpy="0 0 0"/>
         <geometry>
-          <!-- <mesh filename="file://$(find melon_description)/meshes/left_wheel_1.stl" scale="0.001 0.001 0.001"/> -->
           <mesh filename="package://melon_description/meshes/left_wheel_1.stl" scale="0.001 0.001 0.001"/>
         </geometry>
@@ -89,9 +174,6 @@
       </visual>
       <collision>
-        <origin xyz="0.02 0.0 0.0" rpy="0 1.57 0"/>
-        <!-- <origin xyz="-0.277998 0.007002 -0.10065" rpy="0 0 0"/> -->
-        <geometry>
-          <!-- <mesh filename="file://$(find melon_description)/meshes/left_wheel_1.stl" scale="0.001 0.001 0.001"/> -->
-          <!-- <mesh filename="package://melon_description/meshes/left_wheel_1.stl" scale="0.001 0.001 0.001"/> -->
+        <origin xyz="0.01 0.0 0.0" rpy="0 1.57 0"/>
+        <geometry>
           <cylinder length="0.05" radius="0.10065"/>
         </geometry>
@@ -99,25 +181,25 @@
     </link>
     <!-- passive wheel -->
-    <!-- front -->
-    <joint name="${prefix}front_passive_wheel_x_frame_joint" type="continuous">
+    <!-- front left -->
+    <joint name="${prefix}front_left_passive_wheel_x_frame_joint" type="continuous">
       <parent link="${prefix}base_link" />
-      <child link="${prefix}front_passive_wheel_x_frame" />
+      <child link="${prefix}front_left_passive_wheel_x_frame" />
       <axis xyz="1.0 0.0 0.0" />
       <limit effort="1.0" velocity="3.0" />
-      <origin xyz="0.3 0.0 0.025" rpy="0 0 0"/>
-      <dynamics damping="1.0"/>
-    </joint>
-    <link name="${prefix}front_passive_wheel_x_frame">
-      <inertial>
-          <mass value="0.2"/>
-          <origin xyz="0 0 0"/>
-          <inertia ixx="0.001" ixy="0" ixz="0"
-                   iyy="0.001" iyz="0"
-                   izz="0.001"/>
-      </inertial>
-    </link>
-    <joint name="${prefix}front_passive_wheel_y_frame_joint" type="continuous">
-      <parent link="${prefix}front_passive_wheel_x_frame" />
-      <child link="${prefix}front_passive_wheel_y_frame" />
+      <origin xyz="0.3 0.2 0.025" rpy="0 0 0"/>
+      <dynamics damping="1.0"/>
+    </joint>
+    <link name="${prefix}front_left_passive_wheel_x_frame">
+      <inertial>
+          <mass value="0.2"/>
+          <origin xyz="0 0 0"/>
+          <inertia ixx="0.001" ixy="0" ixz="0"
+                   iyy="0.001" iyz="0"
+                   izz="0.001"/>
+      </inertial>
+    </link>
+    <joint name="${prefix}front_left_passive_wheel_y_frame_joint" type="continuous">
+      <parent link="${prefix}front_left_passive_wheel_x_frame" />
+      <child link="${prefix}front_left_passive_wheel_y_frame" />
       <axis xyz="0.0 1.0 0.0" />
       <limit effort="1.0" velocity="3.0" />
@@ -125,16 +207,16 @@
       <dynamics damping="1.0"/>
     </joint>
-    <link name="${prefix}front_passive_wheel_y_frame">
-      <inertial>
-          <mass value="0.2"/>
-          <origin xyz="0 0 0"/>
-          <inertia ixx="0.001" ixy="0" ixz="0"
-                   iyy="0.001" iyz="0"
-                   izz="0.001"/>
-      </inertial>
-    </link>
-    <joint name="${prefix}front_passive_wheel_z_frame_joint" type="continuous">
-      <parent link="${prefix}front_passive_wheel_y_frame" />
-      <child link="${prefix}front_passive_wheel_z_link" />
+    <link name="${prefix}front_left_passive_wheel_y_frame">
+      <inertial>
+          <mass value="0.2"/>
+          <origin xyz="0 0 0"/>
+          <inertia ixx="0.001" ixy="0" ixz="0"
+                   iyy="0.001" iyz="0"
+                   izz="0.001"/>
+      </inertial>
+    </link>
+    <joint name="${prefix}front_left_passive_wheel_z_frame_joint" type="continuous">
+      <parent link="${prefix}front_left_passive_wheel_y_frame" />
+      <child link="${prefix}front_left_passive_wheel_z_link" />
       <axis xyz="0.0 0.0 1.0" />
       <limit effort="1.0" velocity="3.0" />
@@ -142,45 +224,45 @@
       <dynamics damping="1.0"/>
     </joint>
-    <link name="${prefix}front_passive_wheel_z_link">
-      <visual>
-        <geometry>
-          <sphere radius="0.025"/>
-        </geometry>
-        <material name="dark"/>
-      </visual>
-      <collision>
-        <geometry>
-          <sphere radius="0.025"/>
-        </geometry>
-      </collision>
-      <inertial>
-          <mass value="0.2"/>
-          <origin xyz="0 0 0"/>
-          <inertia ixx="0.001" ixy="0" ixz="0"
-                   iyy="0.001" iyz="0"
-                   izz="0.001"/>
-      </inertial>
-    </link>
-    <!-- back -->
-    <joint name="${prefix}back_passive_wheel_x_frame_joint" type="continuous">
+    <link name="${prefix}front_left_passive_wheel_z_link">
+      <visual>
+        <geometry>
+          <sphere radius="0.025"/>
+        </geometry>
+        <material name="dark"/>
+      </visual>
+      <collision>
+        <geometry>
+          <sphere radius="0.025"/>
+        </geometry>
+      </collision>
+      <inertial>
+          <mass value="0.2"/>
+          <origin xyz="0 0 0"/>
+          <inertia ixx="0.001" ixy="0" ixz="0"
+                   iyy="0.001" iyz="0"
+                   izz="0.001"/>
+      </inertial>
+    </link>
+    <!-- front right -->
+    <joint name="${prefix}front_right_passive_wheel_x_frame_joint" type="continuous">
       <parent link="${prefix}base_link" />
-      <child link="${prefix}back_passive_wheel_x_frame" />
+      <child link="${prefix}front_right_passive_wheel_x_frame" />
       <axis xyz="1.0 0.0 0.0" />
       <limit effort="1.0" velocity="3.0" />
-      <origin xyz="-0.33 0.0 0.025" rpy="0 0 0"/>
-      <dynamics damping="1.0"/>
-    </joint>
-    <link name="${prefix}back_passive_wheel_x_frame">
-      <inertial>
-          <mass value="0.2"/>
-          <origin xyz="0 0 0"/>
-          <inertia ixx="0.001" ixy="0" ixz="0"
-                   iyy="0.001" iyz="0"
-                   izz="0.001"/>
-      </inertial>
-    </link>
-    <joint name="${prefix}back_passive_wheel_y_frame_joint" type="continuous">
-      <parent link="${prefix}back_passive_wheel_x_frame" />
-      <child link="${prefix}back_passive_wheel_y_frame" />
+      <origin xyz="0.3 -0.2 0.025" rpy="0 0 0"/>
+      <dynamics damping="1.0"/>
+    </joint>
+    <link name="${prefix}front_right_passive_wheel_x_frame">
+      <inertial>
+          <mass value="0.2"/>
+          <origin xyz="0 0 0"/>
+          <inertia ixx="0.001" ixy="0" ixz="0"
+                   iyy="0.001" iyz="0"
+                   izz="0.001"/>
+      </inertial>
+    </link>
+    <joint name="${prefix}front_right_passive_wheel_y_frame_joint" type="continuous">
+      <parent link="${prefix}front_right_passive_wheel_x_frame" />
+      <child link="${prefix}front_right_passive_wheel_y_frame" />
       <axis xyz="0.0 1.0 0.0" />
       <limit effort="1.0" velocity="3.0" />
@@ -188,16 +270,16 @@
       <dynamics damping="1.0"/>
     </joint>
-    <link name="${prefix}back_passive_wheel_y_frame">
-      <inertial>
-          <mass value="0.2"/>
-          <origin xyz="0 0 0"/>
-          <inertia ixx="0.001" ixy="0" ixz="0"
-                   iyy="0.001" iyz="0"
-                   izz="0.001"/>
-      </inertial>
-    </link>
-    <joint name="${prefix}back_passive_wheel_z_frame_joint" type="continuous">
-      <parent link="${prefix}back_passive_wheel_y_frame" />
-      <child link="${prefix}back_passive_wheel_z_link" />
+    <link name="${prefix}front_right_passive_wheel_y_frame">
+      <inertial>
+          <mass value="0.2"/>
+          <origin xyz="0 0 0"/>
+          <inertia ixx="0.001" ixy="0" ixz="0"
+                   iyy="0.001" iyz="0"
+                   izz="0.001"/>
+      </inertial>
+    </link>
+    <joint name="${prefix}front_right_passive_wheel_z_frame_joint" type="continuous">
+      <parent link="${prefix}front_right_passive_wheel_y_frame" />
+      <child link="${prefix}front_right_passive_wheel_z_link" />
       <axis xyz="0.0 0.0 1.0" />
       <limit effort="1.0" velocity="3.0" />
@@ -205,5 +287,131 @@
       <dynamics damping="1.0"/>
     </joint>
-    <link name="${prefix}back_passive_wheel_z_link">
+    <link name="${prefix}front_right_passive_wheel_z_link">
+      <visual>
+        <geometry>
+          <sphere radius="0.025"/>
+        </geometry>
+        <material name="dark"/>
+      </visual>
+      <collision>
+        <geometry>
+          <sphere radius="0.025"/>
+        </geometry>
+      </collision>
+      <inertial>
+          <mass value="0.2"/>
+          <origin xyz="0 0 0"/>
+          <inertia ixx="0.001" ixy="0" ixz="0"
+                   iyy="0.001" iyz="0"
+                   izz="0.001"/>
+      </inertial>
+    </link>
+    <!-- back left-->
+    <joint name="${prefix}back_left_passive_wheel_x_frame_joint" type="continuous">
+      <parent link="${prefix}base_link" />
+      <child link="${prefix}back_left_passive_wheel_x_frame" />
+      <axis xyz="1.0 0.0 0.0" />
+      <limit effort="1.0" velocity="3.0" />
+      <origin xyz="-0.33 0.2 0.025" rpy="0 0 0"/>
+      <dynamics damping="1.0"/>
+    </joint>
+    <link name="${prefix}back_left_passive_wheel_x_frame">
+      <inertial>
+          <mass value="0.2"/>
+          <origin xyz="0 0 0"/>
+          <inertia ixx="0.001" ixy="0" ixz="0"
+                   iyy="0.001" iyz="0"
+                   izz="0.001"/>
+      </inertial>
+    </link>
+    <joint name="${prefix}back_left_passive_wheel_y_frame_joint" type="continuous">
+      <parent link="${prefix}back_left_passive_wheel_x_frame" />
+      <child link="${prefix}back_left_passive_wheel_y_frame" />
+      <axis xyz="0.0 1.0 0.0" />
+      <limit effort="1.0" velocity="3.0" />
+      <origin xyz="0 0 0" rpy="0 0 0"/>
+      <dynamics damping="1.0"/>
+    </joint>
+    <link name="${prefix}back_left_passive_wheel_y_frame">
+      <inertial>
+          <mass value="0.2"/>
+          <origin xyz="0 0 0"/>
+          <inertia ixx="0.001" ixy="0" ixz="0"
+                   iyy="0.001" iyz="0"
+                   izz="0.001"/>
+      </inertial>
+    </link>
+    <joint name="${prefix}back_left_passive_wheel_z_frame_joint" type="continuous">
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
File: melon_ws/src/melon_description/urdf/materials.xacro (robot description, xacro)
@@ -1,6 +1,12 @@
 <?xml version="1.0" ?>
 <robot xmlns:xacro="http://www.ros.org/wiki/xacro" >
+  <material name="dark_blue">
+    <color rgba="0.0 0.5 0.576 1.0"/>
+  </material>
   <material name="black">
       <color rgba="0.0 0.0 0.0 1.0"/>
+  </material>
+  <material name="dark_black">
+    <color rgba="0.1 0.1 0.1 1.0"/>
   </material>
   <material name="dark">
@@ -16,3 +22,15 @@
     <color rgba="0.10 0.15 0.17 1.0"/>
   </material>
+  <material name="gray_blue">
+    <color rgba="0.271 0.294 0.306 1.0"/>
+  </material>
+  <material name="ocean_blue">
+    <color rgba="0.247 0.400 0.627 1.0"/>
+  </material>
+  <material name="charcoal">
+    <color rgba="0.129 0.129 0.129 1.0"/>
+  </material>
+  <material name="steel_gray">
+    <color rgba="0.325 0.376 0.392 1.0"/>
+  </material>
 </robot>

File: melon_ws/src/melon_description/urdf/melon.urdf (robot description, URDF)
Before this commit: robot Melon, 35 links, 34 joints
Links:
- removed link back_passive_wheel_x_frame
- removed link back_passive_wheel_y_frame
- removed link back_passive_wheel_z_link
- removed link front_passive_wheel_x_frame
- removed link front_passive_wheel_y_frame
- removed link front_passive_wheel_z_link
- added link back_left_passive_wheel_x_frame, mass 0.2
- added link back_left_passive_wheel_y_frame, mass 0.2
- added link back_left_passive_wheel_z_link, mass 0.2; collision sphere radius=0.025; visual sphere radius=0.025
- added link back_right_passive_wheel_x_frame, mass 0.2
- added link back_right_passive_wheel_y_frame, mass 0.2
- added link back_right_passive_wheel_z_link, mass 0.2; collision sphere radius=0.025; visual sphere radius=0.025
- added link front_left_passive_wheel_x_frame, mass 0.2
- added link front_left_passive_wheel_y_frame, mass 0.2
- added link front_left_passive_wheel_z_link, mass 0.2; collision sphere radius=0.025; visual sphere radius=0.025
- added link front_right_passive_wheel_x_frame, mass 0.2
- added link front_right_passive_wheel_y_frame, mass 0.2
- added link front_right_passive_wheel_z_link, mass 0.2; collision sphere radius=0.025; visual sphere radius=0.025
- link base_link: geometry collision mesh filename=package://melon_description/meshes/ballfoint.stl scale=0.001 0.001 0.001; collision mesh filename=package://melon_description/meshes/ballfoint.stl scale=0.001 0.001 0.001
- link base_scan: geometry collision box size=0.11 0.11 0.02; collision cylinder length=0.05 radius=0.05
Joints:
- removed joint back_passive_wheel_x_frame_joint
- removed joint back_passive_wheel_y_frame_joint
- removed joint back_passive_wheel_z_frame_joint
- removed joint front_passive_wheel_x_frame_joint
- removed joint front_passive_wheel_y_frame_joint
- removed joint front_passive_wheel_z_frame_joint
- added joint back_left_passive_wheel_x_frame_joint: type continuous, parent base_link, child back_left_passive_wheel_x_frame, origin xyz=-0.33 0.2 0.025 rpy=0 0 0, axis 1.0 0.0 0.0, limit effort=1.0 velocity=3.0
- added joint back_left_passive_wheel_y_frame_joint: type continuous, parent back_left_passive_wheel_x_frame, child back_left_passive_wheel_y_frame, origin xyz=0 0 0 rpy=0 0 0, axis 0.0 1.0 0.0, limit effort=1.0 velocity=3.0
- added joint back_left_passive_wheel_z_frame_joint: type continuous, parent back_left_passive_wheel_y_frame, child back_left_passive_wheel_z_link, origin xyz=0 0 0 rpy=0 0 0, axis 0.0 0.0 1.0, limit effort=1.0 velocity=3.0
- added joint back_right_passive_wheel_x_frame_joint: type continuous, parent base_link, child back_right_passive_wheel_x_frame, origin xyz=-0.33 -0.2 0.025 rpy=0 0 0, axis 1.0 0.0 0.0, limit effort=1.0 velocity=3.0
- added joint back_right_passive_wheel_y_frame_joint: type continuous, parent back_right_passive_wheel_x_frame, child back_right_passive_wheel_y_frame, origin xyz=0 0 0 rpy=0 0 0, axis 0.0 1.0 0.0, limit effort=1.0 velocity=3.0
- added joint back_right_passive_wheel_z_frame_joint: type continuous, parent back_right_passive_wheel_y_frame, child back_right_passive_wheel_z_link, origin xyz=0 0 0 rpy=0 0 0, axis 0.0 0.0 1.0, limit effort=1.0 velocity=3.0
- added joint front_left_passive_wheel_x_frame_joint: type continuous, parent base_link, child front_left_passive_wheel_x_frame, origin xyz=0.3 0.2 0.025 rpy=0 0 0, axis 1.0 0.0 0.0, limit effort=1.0 velocity=3.0
- added joint front_left_passive_wheel_y_frame_joint: type continuous, parent front_left_passive_wheel_x_frame, child front_left_passive_wheel_y_frame, origin xyz=0 0 0 rpy=0 0 0, axis 0.0 1.0 0.0, limit effort=1.0 velocity=3.0
- added joint front_left_passive_wheel_z_frame_joint: type continuous, parent front_left_passive_wheel_y_frame, child front_left_passive_wheel_z_link, origin xyz=0 0 0 rpy=0 0 0, axis 0.0 0.0 1.0, limit effort=1.0 velocity=3.0
- added joint front_right_passive_wheel_x_frame_joint: type continuous, parent base_link, child front_right_passive_wheel_x_frame, origin xyz=0.3 -0.2 0.025 rpy=0 0 0, axis 1.0 0.0 0.0, limit effort=1.0 velocity=3.0
- added joint front_right_passive_wheel_y_frame_joint: type continuous, parent front_right_passive_wheel_x_frame, child front_right_passive_wheel_y_frame, origin xyz=0 0 0 rpy=0 0 0, axis 0.0 1.0 0.0, limit effort=1.0 velocity=3.0
- added joint front_right_passive_wheel_z_frame_joint: type continuous, parent front_right_passive_wheel_y_frame, child front_right_passive_wheel_z_link, origin xyz=0 0 0 rpy=0 0 0, axis 0.0 0.0 1.0, limit effort=1.0 velocity=3.0
- joint left_wheel_joint: origin xyz=0.007002 0.277998 0.10065 rpy=0 0 1.57 -> xyz=0.007002 0.279998 0.10065 rpy=0 0 1.57
- joint mid_mount_joint: origin xyz=-0.2 0 0.765 rpy=0 0 1.57 -> xyz=0.3 0 0.765 rpy=0 0 1.57
